Commit message: added hande as xml file and abstract simulation class + abstracting more initiated as well as clean up

File: objects/hande/hande.urdf (robot description, URDF)
Before this commit: robot robotiq_hande, 3 links, 2 joints
Links:
- link hand_e_link: geometry collision mesh filename=assets/stl/hand_e.stl scale=1.0 1.0 1.0; visual mesh filename=assets/stl/hand_e.stl scale=1.0 1.0 1.0
- link hande_left_finger: geometry collision mesh filename=assets/stl/finger_1.stl scale=1.0 1.0 1.0; visual mesh filename=assets/stl/finger_1.stl scale=1.0 1.0 1.0
- link hande_right_finger: geometry collision mesh filename=assets/stl/finger_2.stl scale=1.0 1.0 1.0; visual mesh filename=assets/stl/finger_2.stl scale=1.0 1.0 1.0
