Commit message: task board + flexcell load in (some meshes broken - inverted normals) + ros communication

File: objects/hand-e/hand-e.urdf (robot description, URDF)
Before this commit: robot robotiq_hande, 3 links, 2 joints
Links:
- link hand_e_link: geometry collision mesh filename=assets/stl/hand-e.stl scale=1.0 1.0 1.0; visual mesh filename=assets/stl/hand-e.stl scale=1.0 1.0 1.0
